File: elasticNode.brd (EAGLE design)
At the start: 160 x 100 mm, 36 parts, among them U1 TS1102, U2 TS1102, U3 TS1102, U4 74AHC573, U5 SST26VF032B, U6 SST26VF032B

Commit message: working on elastic node
Parts:
- added C25, C26: 22u, passive:0805
- added C27: 10u, passive:0805
- added L1, L2: (no value), passive:0805
- added R5: 6k8, passive:0805
- added R6, R7, R8: 1k5, passive:0805
- added U7: LTC3419, power:MSOP10
Connections:
- removed net RS3+: R3.2, U3.5
- removed net RS3-: R3.1, U3.4
- new net 5V: C27.1, U7.2, U7.3, U7.7
- new net N$1: L2.2, U7.8
- new net N$2: R5.2, R8.2, U7.1
- new net N$7: R6.1, R7.2, U7.10
- new net N$8: L1.1, U7.4
- net 1V2: now also C25.1, L1.2, R6.2
- net 3V3: now also C26.1, L2.1, R3.2, R5.1, U3.5, U7.9
- net GND: now also C25.2, C26.2, C27.2, R7.1, R8.1, U7.5, U7.6
- net MCU_VCC: now also R3.1, U3.4

Commit message: small edits
Parts:
- added R9: (no value), passive:0805
- added U8: TS1102, ic:SOT23
- added U9: MRF24J40MA, wireless:MRF24J40MA
- moved U1 0.12 mm to (24.2, 29.2)
- moved U2 0.12 mm to (24.2, 25.4)
- moved U3 0.12 mm to (24.2, 33.0)
Connections:
- net SENSE_1 renamed SENSE_FPGA_INT
- net SENSE_2 renamed SENSE_FPGA_AUX
- net SENSE_3 renamed SENSE_MCU
- new net SENSE_WIRELESS: U8.3
- new net WIRELESS_CS: U9.8
- new net WIRELESS_INT: U9.4
- new net WIRELESS_RESET: U9.2
- new net WIRELESS_VCC: R9.1, U8.4, U9.10
- new net WIRELESS_WAKE: U9.3
- net 3V3: now also R9.2, U8.5
- net GND: now also U8.1, U8.2, U9.1, U9.11, U9.12
- net MCU_MISO: now also U9.7
- net MCU_MOSI: now also U9.5
- net MCU_SCK: now also U9.6
Routing:
- net SELECTMAP_D3: track 38.0 -> 0.00 mm, vias 1 -> 0
- net SELECTMAP_D2/FPGA_MISO3: track 29.1 -> 0.00 mm, vias 1 -> 0
- net SELECTMAP_D1/FPGA_MISO2: track 26.8 -> 0.00 mm, vias 1 -> 0
- net SELECTMAP_D0/FPGA_MISO1: track 23.2 -> 0.00 mm, vias 1 -> 0

Commit message: home working on elastic node
Parts:
- removed U3, U8: TS1102, ic:SOT23
- added 47K, R14: 15k, passive:0805
- added C28, C30: 100n, passive:0805
- added C29: 10n, passive:0805
- added C31: 4.7u, passive:0805
- added D1, D2: (no value), opto:0805
- added J1: USB_CONN, connectors:USB_MICRO_B
- added L3: 40, passive:0805
- added R10, R11: 270, passive:0805
- added R12, R13: 0.5, passive:0805
- added RESET_FPGA, RESET_MCU: SPST_BUTTON2PIN_SMT, connectors:SPST_2PIN_SMT
- added U10: FT232R, ic:QFN32
- R1: value (none) -> 300
- R2, R3: value (none) -> 0.5
- R9: value (none) -> 2000
- U1, U2: value TS1102 -> PAC1720; device ic:SOT23 -> sensors:VDFN10
- moved R2 16.4 mm to (24.8, 41.5), turned to 270 degrees
- moved U1 11.8 mm to (30.8, 39.0), turned to 0 degrees
- moved R1 8.91 mm to (34.2, 35.5)
- moved R3 6.56 mm to (24.8, 38.8)
- moved R9 5.15 mm to (32.8, 22.2), turned to 180 degrees
- moved U2 4.76 mm to (28.5, 23.2), turned to 0 degrees
- moved C19 2.39 mm to (62.1, 15.5), turned to 0 degrees
- moved C20 2.37 mm to (62.1, 12.8), turned to 0 degrees
- moved C21 2.37 mm to (62.1, 10.1), turned to 0 degrees
Connections:
- removed net PROGRAM_B: U$2.37
- removed net RESET: U$1.20
- removed net SENSE_FPGA_AUX: U2.3
- removed net SENSE_FPGA_INT: U1.3
- removed net SENSE_MCU: U3.3
- removed net SENSE_WIRELESS: U8.3
- new net 12MHZ: U10.22
- new net FPGA_RESET: 47K.1, RESET_FPGA.2, U$2.37
- new net FTDI_RX: U10.2
- new net FTDI_RXLED: R10.1, U10.11
- new net FTDI_TX: U10.30
- new net FTDI_TXLED: R11.1, U10.10
- new net MCU_RESET: R14.1, RESET_MCU.2, U$1.20
- new net N$14: D2.2, R10.2
- new net N$15: D1.2, R11.2
- new net N$16: R9.2, U2.6
- new net N$17: U10.32
- new net N$18: U10.8
- new net N$19: U10.31
- new net N$20: U10.6
- new net N$21: U10.7
- new net N$22: U10.3
- new net N$26: U10.9
- new net N$27: U1.5, U2.5
- new net N$28: R1.2, U1.6
- new net N$3: C28.1, U10.16
- new net N$4: U10.28
- new net N$5: U10.27
- new net N$6: U10.18
- new net SCL: U$1.25
- new net SDA: U$1.26
- new net TWI_CLK: U1.9, U2.9
- new net TWI_DATA: U1.8, U2.8
- new net USBD+: J1.3, U10.14
- new net USBD-: J1.2, U10.15
- new net USB_SHIELD: J1.SHIELD1, J1.SHIELD2
- new net USB_VCC: C30.1, C31.1, L3.2, R12.2, U2.1
- new net USB_VCC_RAW: C29.1, J1.1, L3.1
- net 1V2: now also R13.2, U2.3; no longer R1.2, U1.5
- net 3V3: now also U1.1, U1.10, U1.3, U2.10; no longer R9.2, U2.5, U3.5, U8.5
- net 5V: now also D1.1, D2.1, R12.1, U10.1, U10.19, U2.2
- net FPGA_VCCAUX: now also 47K.2, U1.2; no longer U2.4
- net FPGA_VCCINT: now also R13.1, U2.4; no longer R1.1, U1.4
- net GND: now also C28.2, C29.2, C30.2, C31.2, J1.5, R1.1, R9.1, RESET_FPGA.1, RESET_MCU.1, U10.17, U10.20, U10.24, U10.26, U10.33, U10.4; no longer U1.1, U1.2, U2.1, U2.2, U3.1, U3.2, U8.1, U8.2
- net MCU_VCC: now also R14.2, U1.4; no longer U3.4
- net SELECTMAP_D0/FPGA_MISO1: no longer U$1.32
- net SELECTMAP_D1/FPGA_MISO2: no longer U$1.31
- net SELECTMAP_D2/FPGA_MISO3: no longer U$1.30
- net SELECTMAP_D3: no longer U$1.29
- net SELECTMAP_D4: no longer U$1.28
- net SELECTMAP_D5: no longer U$1.27
- net SELECTMAP_D6: no longer U$1.26
- net SELECTMAP_D7: no longer U$1.25
- net WIRELESS_VCC: no longer R9.1, U8.4

Commit message: small routing at home
Parts:
- removed R4: 10k, passive:0805
- U7: value LTC3419 -> LTC3419DFN; device power:MSOP10 -> power:DFN8
- moved C11 25.9 mm to (92.5, 30.4), turned to 90 degrees
- moved C12 22.4 mm to (90.0, 30.4), turned to 90 degrees
- moved U5 16.2 mm to (71.6, 13.4), flipped to the top, turned to 180 degrees
- moved U9 15.1 mm to (122.0, 43.2), flipped to the top, turned to 0 degrees
- moved C26 14.8 mm to (20.2, 54.5), turned to 0 degrees
- moved L1 12.5 mm to (28.0, 48.8)
- moved L2 12.3 mm to (19.0, 48.8)
- moved R5 10.3 mm to (20.0, 52.0), turned to 0 degrees
- moved R8 8.96 mm to (22.0, 50.5)
- moved C27 7.26 mm to (24.4, 45.5), turned to 180 degrees
- moved U6 7.15 mm to (111.5, 23.9), turned to 90 degrees
- moved C5 6.40 mm to (69.7, 58.5)
- moved C6 6.21 mm to (69.7, 56.2)
- moved C7 6.02 mm to (69.7, 53.9)
- moved C8 6.02 mm to (69.7, 51.4)
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Connections:
- removed net FPGA_SCK: U5.6
- removed net MCU_CE: R4.1, U6.1
- new net MCU_FLASH_CE: U$1.14, U6.1
- new net N$10: U$2.95
- new net N$34: U$2.87
- new net N$35: U$2.88
- new net N$36: U$2.92
- new net N$37: U$2.93
- new net N$38: U$2.94
- new net N$46: U$2.121
- new net SUSPEND: U$2.73
- net 3V3: now also U7.7; no longer U7.9
- net 5V: now also U7.5; no longer U7.7
- net A0: now also U$2.111
- net A1: now also U$2.112
- net A10: now also U$2.80
- net A11: now also U$2.81
- net A12: now also U$2.82
- net A13: now also U$2.83
- net A14: now also U$2.84
- net A15: now also U$2.85
- net A2: now also U$2.114
- net A3: now also U$2.115
- net A4: now also U$2.116
- net A5: now also U$2.117
- net A6: now also U$2.118
- net A7: now also U$2.119
- net A8: now also U$2.78
- net A9: now also U$2.79
- net AD0: now also U$2.97
- net AD1: now also U$2.98
- net AD2: now also U$2.99
- net AD3: now also U$2.100
- net AD4: now also U$2.101
- net AD5: now also U$2.102
- net AD6: now also U$2.104
- net AD7: now also U$2.105
- net ALE: now also U$2.120
- net CCLK: now also U5.6
- net GND: now also U10.P$1, U10.P$2, U10.P$3, U10.P$4, U10.P$5, U10.P$6, U10.P$7, U10.P$8, U10.P$9, U7.9; no longer U7.5, U7.6
- net MCU_VCC: no longer R4.2
- net N$1: now also U7.4; no longer U7.8
- net N$27: now also U1.P$1, U1.P$2, U1.P$3, U1.P$4, U2.P$1, U2.P$2, U2.P$3, U2.P$4
- net N$7: now also U7.8; no longer U7.10
- net N$8: now also U7.6; no longer U7.4
- net RD: now also U$2.75
- net WIRELESS_CS: now also U$1.15
- net WIRELESS_INT: now also U$1.9
- net WIRELESS_RESET: now also U$1.7
- net WIRELESS_WAKE: now also U$1.8
- net WR: now also U$2.74
Routing:
- net ALE: track 0.00 -> 41.7 mm, vias 0 -> 1
- net MCU_MISO: track 0.00 -> 36.4 mm, vias 0 -> 1
- net WIRELESS_CS: track 0.00 -> 34.9 mm, vias 0 -> 1
- net CSO_B: track 0.00 -> 25.8 mm
- net MCU_MOSI: track 0.00 -> 25.7 mm, vias 0 -> 1
- net AD0: track 0.00 -> 24.5 mm, vias 0 -> 1
- net WIRELESS_RESET: track 0.00 -> 24.5 mm, vias 0 -> 1
- net AD5: track 0.00 -> 24.3 mm, vias 0 -> 1
- net AD4: track 0.00 -> 23.4 mm, vias 0 -> 1
- net AD3: track 0.00 -> 23.2 mm, vias 0 -> 1
- net AD1: track 0.00 -> 23.2 mm, vias 0 -> 1
- net AD6: track 0.00 -> 22.8 mm, vias 0 -> 1
- net WIRELESS_WAKE: track 0.00 -> 22.7 mm, vias 0 -> 1
- net AD7: track 0.00 -> 22.6 mm, vias 0 -> 1
- net AD2: track 0.00 -> 21.9 mm, vias 0 -> 1
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- added copper zone on layer 1, net 1V2
- added copper zone on layer 1, net 3V3
- added copper zone on layer 1, net 5V
- added copper zone on layer 1, net N$1
- added copper zone on layer 1, net N$8

Commit message: lots of routing, and reorganising
Parts:
- added U$3: ISP_CONN_6PIN, connectors:3X2_HEADER_SMT
- added U$4: FTDI_CONN_6PINSMT_KEEPOUT, connectors:6X1_FTDI_SMT
- moved J1 131.3 mm to (133.5, 16.5), turned to 90 degrees
- moved C31 120.1 mm to (127.2, 10.8), turned to 270 degrees
- moved C28 119.9 mm to (127.9, 18.7), turned to 270 degrees
- moved C29 119.3 mm to (127.2, 13.8), turned to 270 degrees
- moved C30 115.2 mm to (124.8, 10.8), turned to 270 degrees
- moved U10 114.1 mm to (125.0, 22.8), turned to 0 degrees
- moved L3 113.1 mm to (124.2, 14.8), turned to 180 degrees
- moved D2 107.2 mm to (121.2, 14.5), turned to 90 degrees
- moved R10 106.7 mm to (121.2, 17.5), turned to 270 degrees
- moved C25 106.0 mm to (131.8, 38.2)
- moved C26 106.0 mm to (125.0, 38.2)
- moved L1 106.0 mm to (132.8, 32.5)
- moved L2 106.0 mm to (123.8, 32.5)
- moved R5 106.0 mm to (124.8, 35.8)
- moved R6 106.0 mm to (131.8, 35.8)
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Connections:
- removed net FPGA_MISO0: U$2.64, U5.5
- removed net FTDI_RX: U10.2
- removed net FTDI_TX: U10.30
- removed net N$10: U$2.95
- removed net N$27: U1.5, U1.P$1, U1.P$2, U1.P$3, U1.P$4, U2.5, U2.P$1, U2.P$2, U2.P$3, U2.P$4
- removed net N$38: U$2.94
- removed net SCL: U$1.25
- removed net SDA: U$1.26
- removed net SELECTMAP_D4: U$2.45
- removed net SELECTMAP_D5: U$2.44
- removed net SELECTMAP_D6: U$2.43
- removed net SELECTMAP_D7: U$2.48
- removed net TWI_CLK: U1.9, U2.9
- removed net TWI_DATA: U1.8, U2.8
- new net CSI_B/FPGA_MISO0: U$1.18, U$2.64, U5.5
- new net CTS: U$4.2
- new net MCU_RX0: U$1.2, U$2.94, U$4.4, U10.30
- new net MCU_TX0: U$1.3, U$2.95, U$4.5, U10.2
- new net RTS: U$4.6
- new net SELECTMAP_D4/MCU_TX1: U$1.28, U$2.45
- new net SELECTMAP_D5/MCU_RX1: U$1.27, U$2.44
- new net SELECTMAP_D6/SDA: U$1.26, U$2.43, U1.8, U2.8
- new net SELECTMAP_D7/SCL: U$1.25, U$2.48, U1.9, U2.9
- net 3V3: now also U$3.2, U$4.3
- net CCLK: now also U$1.19
- net GND: now also U$3.6, U$4.1, U1.5, U1.P$1, U1.P$2, U1.P$3, U1.P$4, U2.5, U2.P$1, U2.P$2, U2.P$3, U2.P$4
- net INIT_B: now also U$1.17
- net MCU_MISO: now also U$3.1
- net MCU_MOSI: now also U$3.4
- net MCU_RESET: now also U$3.5
- net MCU_SCK: now also U$3.3
- net SELECTMAP_D0/FPGA_MISO1: now also U$1.32
- net SELECTMAP_D1/FPGA_MISO2: now also U$1.31
- net SELECTMAP_D2/FPGA_MISO3: now also U$1.30
- net SELECTMAP_D3: now also U$1.29
- net WIRELESS_CS: now also U$1.6; no longer U$1.15
Routing:
- net INIT_B: track 0.00 -> 46.8 mm, vias 0 -> 3
- net SELECTMAP_D7/SCL: track 0.00 -> 40.2 mm, vias 0 -> 1
- net SELECTMAP_D6/SDA: track 0.00 -> 39.7 mm, vias 0 -> 1
- net CSI_B/FPGA_MISO0: track 0.00 -> 38.6 mm, vias 0 -> 3
- net SELECTMAP_D5/MCU_RX1: track 0.00 -> 38.4 mm, vias 0 -> 1
- net SELECTMAP_D4/MCU_TX1: track 0.00 -> 36.9 mm, vias 0 -> 1
- net SELECTMAP_D3: track 0.00 -> 35.4 mm, vias 0 -> 1
- net CCLK: track 15.4 -> 43.9 mm, vias 0 -> 3
- net MCU_RX0: track 0.00 -> 25.1 mm, vias 0 -> 1
- net SELECTMAP_D2/FPGA_MISO3: track 10.8 -> 35.7 mm, vias 0 -> 1
- net SELECTMAP_D1/FPGA_MISO2: track 14.0 -> 37.3 mm, vias 0 -> 1
- net MCU_TX0: track 0.00 -> 22.7 mm, vias 0 -> 1
- net MCU_SCK: track 20.2 -> 41.6 mm
- net MCU_RESET: track 10.2 -> 30.8 mm, vias 0 -> 1
- net SELECTMAP_D0/FPGA_MISO1: track 10.8 -> 31.2 mm, vias 0 -> 1
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
Commit message: small home edits
Routing:
- net 5V: track 0.00 -> 4.16 mm, vias 0 -> 2
- net N$8: track 0.00 -> 3.56 mm
- net 3V3: track 0.00 -> 2.11 mm, vias 0 -> 4
- added copper zone on layer 2, net 1V2
- added copper zone on layer 3, net 3V3
- added copper zone on layer 1, net GND
- added copper zone on layer 16, net GND

Commit message: lots of routing, removed latch
Parts:
- removed 47K: 15k, passive:0805
- removed U4: 74AHC573, ic:SOIC20
- added J2: FEMALE_HEADER_5X2, connectors:5X2_HEADER
- added J3, J4: FEMALE_HEADER_2X1, connectors:2X1_HEADER
- added J5: JTAG_CONN_6PINTHT, connectors:6X1_HEADER
- added J6: FEMALE_HEADER_2X2, connectors:2X2_HEADER
- added R15: 15k, passive:0805
- added R16, R17: 2.4k, passive:0805
- added R18, R4: 1.5k, passive:0805
- U$1: value ATMEGA64A -> ATMEGA64AQFN; device ic:TQFP64 -> ic:QFN64
- U$4: value FTDI_CONN_6PINSMT_KEEPOUT -> SPST_DIP_2SMT; device connectors:6X1_FTDI_SMT -> connectors:SPST_DIP2_SMT
- moved C5 46.1 mm to (61.1, 13.2)
- moved C6 41.6 mm to (61.1, 15.5)
- moved U9 28.3 mm to (94.5, 46.5)
- moved U$4 24.6 mm to (89.8, 15.8), turned to 0 degrees
- moved C25 17.8 mm to (114.0, 37.5)
- moved C26 17.8 mm to (107.2, 37.5)
- moved L1 17.8 mm to (115.0, 31.8)
- moved L2 17.8 mm to (106.0, 31.8)
- moved R5 17.8 mm to (107.0, 35.0)
- moved R6 17.8 mm to (114.0, 35.0)
- moved R7 17.8 mm to (111.2, 35.0)
- moved R8 17.8 mm to (109.0, 33.5)
- moved U7 17.8 mm to (110.2, 31.2)
- moved C27 17.8 mm to (111.5, 28.5)
- moved C28 10.0 mm to (117.9, 18.9)
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Connections:
- removed net A0: U$2.111, U4.19
- removed net A1: U$2.112, U4.18
- removed net A2: U$2.114, U4.17
- removed net A3: U$2.115, U4.16
- removed net A4: U$2.116, U4.15
- removed net A5: U$2.117, U4.14
- removed net A6: U$2.118, U4.13
- removed net A7: U$2.119, U4.12
- removed net CTS: U$4.2
- removed net FTDI_TXLED: R11.1, U10.10
- removed net N$15: D1.2, R11.2
- removed net N$46: U$2.121
- removed net RTS: U$4.6
- removed net TCK: U$2.109
- removed net TDI: U$2.110
- removed net TDO: U$2.106
- removed net TMS: U$2.107
- new net FPGA_GPIO_0: J2.10, U$2.1
- new net FPGA_GPIO_1: J2.1, U$2.2
- new net FPGA_GPIO_2: J2.9, U$2.5
- new net FPGA_GPIO_3: J2.2, U$2.6
- new net FPGA_GPIO_4: J2.8, U$2.7
- new net FPGA_GPIO_5: J2.3, U$2.8
- new net FPGA_GPIO_6: J2.7, U$2.9
- new net FPGA_GPIO_7: J2.4, U$2.10
- new net FPGA_GPIO_8: J2.6, U$2.11
- new net FPGA_GPIO_9: J2.5, U$2.12
- new net JTAG_TCK: J5.P$3, U$1.57, U$2.109
- new net JTAG_TDI: J5.P$5, U$1.55, U$2.110
- new net JTAG_TDO: J5.P$4, U$1.56, U$2.106
- new net JTAG_TMS: J5.P$6, U$1.54, U$2.107
- new net MCU_GPIO_0: J6.1, U$1.58
- new net MCU_GPIO_1: J6.4, U$1.59
- new net MCU_GPIO_2: J6.3, U$1.60
- new net MCU_GPIO_3: J6.2, U$1.61
- new net N$10: R11.2, U10.10
- new net N$11: D1.2, R11.1
- net 3V3: no longer U$4.3
- net AD0: now also U$2.105; no longer U$2.97, U4.2
- net AD1: now also U$2.104; no longer U$2.98, U4.3
- net AD2: now also U$2.102; no longer U$2.99, U4.4
- net AD3: now also U$2.101; no longer U$2.100, U4.5
- net AD4: now also U$2.100; no longer U$2.101, U4.6
- net AD5: now also U$2.99; no longer U$2.102, U4.7
- net AD6: now also U$2.98; no longer U$2.104, U4.8
- net AD7: now also U$2.97; no longer U$2.105, U4.9
- net ALE: now also U$2.95; no longer U$2.120, U4.11
- net FPGA_RESET: now also R15.1; no longer 47K.1
- net FPGA_VCCAUX: now also J4.1, J5.P$1, R15.2, R16.1, R17.1; no longer 47K.2
- net FPGA_VCCINT: now also J3.1
- net GND: now also J3.3, J4.3, J5.P$2, R18.1, R4.2, U$1.PAD, U$1.VIA1, U$1.VIA2, U$1.VIA3, U$1.VIA4, U$1.VIA5, U$1.VIA6, U$1.VIA7, U$1.VIA8, U$1.VIA9, U$4.3, U$4.4; no longer U$4.1, U4.1, U4.10
- net MCU_RX0: no longer U$2.94, U$4.4
- net MCU_TX0: no longer U$2.95, U$4.5
- net MCU_VCC: no longer U4.20
- net MODE0: now also R16.2, U$4.1
- net MODE1: now also R17.2, U$4.2
- net SELECTMAP_D6/SDA: now also R18.2
- net SELECTMAP_D7/SCL: now also R4.1
- net USB_SHIELD: no longer J1.SHIELD2
Routing:
- net FPGA_VCCAUX: track 0.00 -> 124.0 mm, vias 0 -> 16
- net 3V3: track 2.11 -> 53.2 mm, vias 4 -> 6
- net SELECTMAP_D7/SCL: track 40.2 -> 88.6 mm, vias 1 -> 3
- net 5V: track 4.16 -> 52.1 mm, vias 2 -> 5
- net SELECTMAP_D6/SDA: track 39.7 -> 85.6 mm, vias 1 -> 2
- net FPGA_VCCINT: track 0.00 -> 35.8 mm, vias 0 -> 6
- net ALE: track 41.7 -> 9.50 mm
- net MCU_VCC: track 0.00 -> 29.2 mm, vias 0 -> 7
- net JTAG_TCK: track 0.00 -> 27.0 mm
- net JTAG_TDO: track 0.00 -> 26.5 mm
- net MCU_GPIO_1: track 0.00 -> 25.6 mm
- net MODE1: track 0.00 -> 25.5 mm
- net MCU_GPIO_2: track 0.00 -> 25.1 mm
- net MCU_GPIO_0: track 0.00 -> 23.6 mm
- net JTAG_TDI: track 0.00 -> 22.8 mm
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- added copper zone on layer 3, net FPGA_VCCAUX
- added copper zone on layer 2, net FPGA_VCCINT
- added copper zone on layer 3, net MCU_VCC
Other:
- board size 160 x 100 mm -> 82.2 x 52.5 mm
- board text removed: "analog gnd"

Commit message: added another measurement
Parts:
- added D10, D3, D4, D5, D6, D7, D8, D9: (no value), opto:0805
- added J7: FEMALE_HEADER_5X2, connectors:5X2_HEADER
- added R19, R20, R21, R22, R23, R24, R25, R26: (no value), passive:0805
- added R27: 2000, passive:0805
- added R29: 0.5, passive:0805
- added U3: PAC1720, sensors:VDFN10
- added X1: 50MHz, passive:3.2X2.5_OSC
- added X2: 32MHz, passive:3.2X2.5_OSC
- moved C11 49.6 mm to (43.2, 24.8), turned to 270 degrees
- moved C12 49.4 mm to (41.0, 24.8), turned to 270 degrees
- moved C22 47.3 mm to (6.50, 25.5)
- moved C23 47.3 mm to (4.25, 25.5)
- moved C24 47.3 mm to (2.00, 25.5)
- moved C13 45.3 mm to (19.5, 42.8)
- moved C14 45.3 mm to (19.5, 45.0)
- moved C15 45.3 mm to (19.5, 47.2)
- moved RESET_FPGA 45.2 mm to (9.00, 3.75)
- moved C1 45.1 mm to (8.75, 28.2), turned to 270 degrees
- moved C2 45.1 mm to (6.50, 28.2), turned to 270 degrees
- moved C3 45.1 mm to (4.25, 28.2), turned to 270 degrees
- moved C4 45.1 mm to (2.00, 28.2), turned to 270 degrees
- moved J2 44.6 mm to (3.75, 36.8)
- moved C16 44.5 mm to (43.2, 27.8)
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Connections:
- new net FPGA_GPIO_10: J7.10, U$2.24
- new net FPGA_GPIO_11: J7.1, U$2.23
- new net FPGA_GPIO_12: J7.9, U$2.27
- new net FPGA_GPIO_13: J7.2, U$2.26
- new net FPGA_GPIO_14: J7.8, U$2.30
- new net FPGA_GPIO_15: J7.3, U$2.29
- new net FPGA_GPIO_16: J7.7, U$2.33
- new net FPGA_GPIO_17: J7.4, U$2.32
- new net FPGA_GPIO_18: J7.6, U$2.35
- new net FPGA_GPIO_19: J7.5, U$2.34
- new net FPGA_LED0: R19.1, U$2.144
- new net FPGA_LED1: R20.1, U$2.143
- new net FPGA_LED2: R21.1, U$2.142
- new net FPGA_LED3: R22.1, U$2.141
- new net MCU_LED0: R23.1, U$1.16
- new net MCU_LED1: R24.1, U$1.15
- new net MCU_LED2: R25.1, U$1.4
- new net MCU_LED3: R26.1, U$1.5
- new net N$13: D10.1, R26.2
- new net N$15: D9.1, R25.2
- new net N$23: D8.1, R24.2
- new net N$24: D7.1, R23.2
- new net N$25: D6.1, R22.2
- new net N$27: D5.1, R21.2
- new net N$29: D4.1, R20.2
- new net N$30: D3.1, R19.2
- new net N$31: U$2.140
- new net N$32: R27.2, U3.6
- new net OSC_32: U$2.94, X2.3
- new net OSC_50: U$2.131, X1.3
- net 3V3: now also R29.2, U3.10, U3.3
- net 5V: now also R12.2, U2.1; no longer R12.1, U2.2
- net FPGA_VCCAUX: now also X1.1, X1.4, X2.1, X2.4
- net GND: now also D10.2, D3.2, D4.2, D5.2, D6.2, D7.2, D8.2, D9.2, R27.1, R8.2, U3.5, U3.P$1, U3.P$2, U3.P$3, U3.P$4, X1.2, X2.2; no longer R8.1
- net N$2: now also R8.1; no longer R8.2
- net SELECTMAP_D6/SDA: now also U3.8
- net SELECTMAP_D7/SCL: now also U3.9
- net USB_VCC: now also R12.1, U2.2; no longer R12.2, U2.1
- net WIRELESS_VCC: now also R29.1, U3.4
Routing:
- net SELECTMAP_D7/SCL: track 88.6 -> 129.7 mm, vias 3 -> 5
- net SELECTMAP_D6/SDA: track 85.6 -> 125.8 mm, vias 2 -> 4
- net MCU_LED3: track 0.00 -> 37.5 mm, vias 0 -> 2
- net MCU_LED1: track 0.00 -> 36.1 mm, vias 0 -> 2
- net MCU_LED0: track 0.00 -> 35.6 mm, vias 0 -> 2
- net MCU_LED2: track 0.00 -> 34.6 mm, vias 0 -> 2
- net WIRELESS_VCC: track 0.00 -> 23.0 mm
- net FPGA_VCCAUX: track 124.0 -> 141.8 mm, vias 16 -> 18
- net FPGA_GPIO_19: track 0.00 -> 16.8 mm
- net 3V3: track 53.2 -> 69.2 mm, vias 6 -> 8
- net FPGA_GPIO_17: track 0.00 -> 15.3 mm
- net FPGA_GPIO_18: track 0.00 -> 14.0 mm
- net FPGA_GPIO_15: track 0.00 -> 14.0 mm
- net FPGA_GPIO_16: track 0.00 -> 12.5 mm
- net FPGA_GPIO_13: track 0.00 -> 12.4 mm
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