File: elasticNode.sch (EAGLE design)
At the start: 136 parts, among them J1 FEMALE_HEADER_2X1, J2 JUMPER, J3 JUMPER, J5 FEMALE_HEADER_10X2, J6 USB_CONNMICRO_SMT, J7 USB_CONNMICRO_SMT, M1 SISS23DN, M2 SISS23DN, M3 SISS23DN, M4 SISS23DN, U1 AT90USB128, U10 LTC3419DFN, U11 PAC1720, U14 LTC3419DFN, U2 IS66WV51216EALL, U3 MRF24J40MA, U4 SPARTAN7-LX15, U5 ATMEGA32U4QFN, U6 SST26VF032BWDFN, U7 PAC1720, U8 PAC1720, U9 PAC1720, X1 8MHz, X2 50MHz, X3 32MHz, X4 100MHz, X5 8MHz

Commit message: finish the work.
Connections:
- removed net N$1: OUT1.9
- removed net N$31: OUT1.8
- removed net N$32: OUT1.7
- removed net N$33: OUT1.6
- removed net N$8: OUT1.10
- net AD0/SELECTMAP_D7: now also OUT1.10
- net AD1/SELECTMAP_D6: now also OUT1.9
- net AD2/SELECTMAP_D5/MCU_RX1: now also OUT1.6
- net AD3/SELECTMAP_D4/MCU_TX1: now also OUT1.7
- net AD4/SELECTMAP_D3/FPGA_HOLD: now also OUT1.8
- net AD5/SELECTMAP_D2/FPGA_WP: now also OUT1.5
- net AD6/SELECTMAP_D1/SPI_MISO/MCU_PDO: now also OUT1.4
- net AD7/SELECTMAP_D0/SPI_MOSI/PDI: now also OUT1.3
- net ALE/HWB: now also U4.IO_L12P_T1_MRCC_14; no longer U4.IO_L9P_T1_DQS_14
- net FPGA_GPIO_0: now also U4.IO_L14N_T2_SRCC_14; no longer U4.IO_L13N_T2_MRCC_14
- net FPGA_GPIO_1: now also U4.IO_L16N_T2_D31_14; no longer U4.IO_L15N_T2_DQS_DOUT_CSO_B_14
- net FPGA_GPIO_11: now also U4.IO_L17N_T2_D29_14; no longer U4.IO_L18P_T2_D28_14
- net FPGA_GPIO_13: now also U4.IO_L17P_T2_D30_14; no longer U4.IO_L18N_T2_D27_14
- net FPGA_GPIO_14: now also U4.IO_L19N_T3_D25_VREF_14; no longer U4.IO_L19P_T3_D26_14
- net FPGA_GPIO_16: now also U4.IO_L19P_T3_D26_14
- net FPGA_GPIO_18: now also U4.IO_L15N_T2_DQS_DOUT_CSO_B_14; no longer U4.IO_L16N_T2_D31_14
- net FPGA_GPIO_3: now also U4.IO_L21N_T3_DQS_D22_14; no longer U4.IO_L20N_T3_D23_14
- net FPGA_GPIO_4: now also U4.IO_L13N_T2_MRCC_14; no longer U4.IO_L14N_T2_SRCC_14
- net FPGA_GPIO_5: now also U4.IO_L20N_T3_D23_14; no longer U4.IO_L21N_T3_DQS_D22_14
- net FPGA_GPIO_6: now also U4.IO_L18P_T2_D28_14; no longer U4.IO_L17P_T2_D30_14
- net FPGA_GPIO_8: now also U4.IO_L18N_T2_D27_14; no longer U4.IO_L17N_T2_D29_14
- net SRAM_A0: now also U4.IO_L3P_T0_DQS_34; no longer U4.IO_L5P_T0_34
- net SRAM_A1: now also U4.IO_L5P_T0_34; no longer U4.IO_L3P_T0_DQS_34
- net SRAM_CS: now also U4.IO_L1N_T0_34; no longer U4.IO_L6N_T0_VREF_34
- net SRAM_D0: now also U4.IO_L6N_T0_VREF_34; no longer U4.IO_L1N_T0_34
- net SRAM_D6: now also U4.IO_L14P_T2_SRCC_34; no longer U4.IO_L13P_T2_MRCC_34
- net SRAM_D7: now also U4.IO_L13N_T2_MRCC_34; no longer U4.IO_L14P_T2_SRCC_34
- net SRAM_WE: now also U4.IO_L13P_T2_MRCC_34; no longer U4.IO_L13N_T2_MRCC_34
- net XMEM_A10: now also OUT2.1, U4.IO_L10N_T1_D15_14; no longer U4.IO_L7N_T1_D10_14
- net XMEM_A11: now also OUT2.6, U4.IO_L7N_T1_D10_14; no longer U4.IO_L10N_T1_D15_14
- net XMEM_A12: now also OUT2.5, U4.IO_L9N_T1_DQS_D13_14; no longer U4.IO_L7P_T1_D09_14
- net XMEM_A13: now also OUT2.4
- net XMEM_A14: now also OUT2.3, U4.IO_L7P_T1_D09_14; no longer U4.IO_L9N_T1_DQS_D13_14
- net XMEM_A15: now also OUT2.2, U4.IO_L9P_T1_DQS_14; no longer U4.IO_L12P_T1_MRCC_14
- net XMEM_A9: now also U4.IO_L8P_T1_D11_14; no longer U4.IO_L11P_T1_SRCC_14
- net XMEM_RD: now also U4.IO_L11P_T1_SRCC_14; no longer U4.IO_L8P_T1_D11_14
