File: v3/elasticNode.brd (EAGLE design)
At the start: 58.2 x 52.5 mm, 117 parts, among them J1 FEMALE_HEADER_2X1, J2 JUMPER, J3 ISP_CONN_6PIN, J4 FEMALE_HEADER_3X2, J5 FEMALE_HEADER_10X2, J6 USB_CONNMICRO_SMT, M1 SISS23DN, M2 SISS23DN, M3 SISS23DN, U1 AT90USB128, U10 LTC3419DFN, U11 PAC1720, U12 MT41J128M8, U14 LTC3419DFN, U2 ATMEGA64AQFN, U3 MRF24J40MA, U4 SPARTAN7-LX15, U6 SST26VF032BWDFN, U7 PAC1720, U8 PAC1720, U9 PAC1720, X1 8MHz, X2 50MHz, X3 32MHz, X4 100MHz

Commit message: partial v3
Parts:
- removed 1000: 6k8, passive:0805
- removed 2.2K, R37, R38, R39: 1k5, passive:0805
- removed D10: RED, opto:0805
- removed L5, L6: 3.3uH, passive:0805
- removed M3: SISS23DN, power:POWERPAK1212-8
- removed R40: 270, passive:0805
- removed R41, R42: 10k, passive:0805
- removed R43: .8, passive:0805
- removed R44: 240%1, passive:0805
- removed R45: 80.6, passive:0805
- removed TP1, TP2, TP3, TP4, TP5, TP6: TEST_POINTTHT, connectors:THT
- removed U12: MT41J128M8, ic:FBGA78DA
- removed U14: LTC3419DFN, power:DFN8
- added 15K: 10k, passive:0805
- added C20, C23: 4.7uF, passive:0805
- added C21, C22: .47uF, passive:0402
- added C24: .47uF, passive:0805
- added C25: 10n, passive:0805
- added C29, C31: 22u, passive:0805
- added C30: 10u, passive:0805
- added C32: 1u, passive:0805
- added C33, C34: 20pF, passive:0805
- added C35, C36: 20p, passive:0805
- added J10: ISP_CONN_6PIN, connectors:3X2_HEADER_SMT
- added J8, J9: USB_CONNSMT, connectors:USB_MICRO_B_SMT
- added L3: 3.3uH, passive:0805
- added RX: ORANGE, opto:0805
- added S4: SPST_BUTTON2PIN_SMT, connectors:SPST_2PIN_SMT
- added TX: ORANGE 2V, opto:0805
- added U5: SST26VF032B, ic:SOIC8
- C1: value (none) -> 4.7uF
- C10, C15: value 4.7u -> 4.7uF
- C11: value 0.47u -> .47uF; device passive:0805 -> passive:0402
- C12, C18: value 10u -> .47uF; device passive:0805 -> passive:0402
- C13: value 10u -> 0.47uF; device passive:0805 -> passive:0402
- C14: value 0.47u -> 4.7uF
- C16: value 2.2u -> 4.7uF
- C17: value 22u -> 4.7uF
- C19: value 22u -> .47uF; device passive:0805 -> passive:0402
- C2, C3: value 20p -> 4.7uF
- C26: value 22u -> 100n
- C27: value 22u -> 4.7u
- C28: value 10u -> 100n
- C4, C6: value 100u -> 4.7uF; device passive:1210 -> passive:0805
- C5: value 47u -> 4.7uF; device passive:1210 -> passive:0805
- C7: value 47u -> .47uF; device passive:1210 -> passive:0402
- C8: value 4.7 -> .47uF; device passive:0805 -> passive:0402
- C9: value 10u -> 4.7uF
- J1: value FEMALE_HEADER_2X1 -> ISP_CONN_6PIN; device connectors:2X1_HEADER -> connectors:3X2_HEADER_SMT
- J2: value JUMPER -> FEMALE_HEADER_2X2; device connectors:JUMPER_SMT -> connectors:2X2_HEADER
- J3: value ISP_CONN_6PIN -> FEMALE_HEADER_2X1; device connectors:ICSP_SMT -> connectors:2X1_HEADER
- J4: value FEMALE_HEADER_3X2 -> FEMALE_HEADER_2X1; device connectors:3X2_HEADER_SMT -> connectors:2X1_HEADER
- J6: value USB_CONNMICRO_SMT -> FEMALE_HEADER_2X1; device connectors:USB_MICRO_B_SMT -> connectors:2X1_HEADER
- L1: value 3.3uH -> 40Ohm 1.5A
- R1, R2: value 22 -> 2.4k
- R10: value 4.7k -> 750
- R12, R13, R14: value 750 -> 2.4k
- R16: value 2.4k -> 0.8
- R17, R19: value 2.4k -> .8
- R18: value 2.4k -> 0.16
- R20: value 0.8 -> 100
- R21: value .8 -> 300
- R23: value 0.8 -> 2000
- R24, R25: value .8 -> 1.5k
- R26: value 100 -> 1.5k
- R27: value 2000 -> 1.5k
- R28: value 300 -> 6k8
- R29, R30: value 1.5k -> 1k5
- R3: value 2.4k -> 550
- R31: value 6k8 -> 1k5
- R32: value 1k5 -> 270
- R33: value 270 -> 22
- R34: value 1k5 -> 22
- R35: value 750 -> 15k
- R36: value 0.15 -> .8
- R4: value 10k -> 550
- R7: value 550 -> 15k
- R8: value 550 -> 750
- R9: value 15k -> 750
- U1: value AT90USB128 -> ATMEGA64AQFN
- U11: value PAC1720 -> ATMEGA32U4; device sensors:VDFN10 -> ic:QFN44
- U2: value ATMEGA64AQFN -> SST26VF032B; device ic:QFN64 -> ic:SOIC8
- U4: value SPARTAN7-LX15 -> SPARTAN6-LX9; device fpga:FTGB196 -> fpga:TQG144
- U6: value SST26VF032BWDFN -> PAC1720; device ic:WDFN8 -> sensors:VDFN10
- U9: value PAC1720 -> FT232RSSOP28; device sensors:VDFN10 -> ic:SSOP28
- X1: value 8MHz -> 12MHz
- X4: value 100MHz -> 12MHz
- moved R36 106.3 mm to (50.5, 22.5), flipped to the bottom, turned to 180 degrees
- moved C28 83.1 mm to (3.50, 32.0), flipped to the bottom, turned to 180 degrees
- moved R35 81.1 mm to (41.5, 5.50), turned to 180 degrees
- moved U11 79.3 mm to (17.2, 14.5), flipped to the bottom, turned to 90 degrees
- moved C26 75.1 mm to (12.8, 26.0), flipped to the bottom, turned to 90 degrees
- moved C27 75.0 mm to (15.0, 26.0), flipped to the bottom, turned to 90 degrees
- moved U7 60.3 mm to (45.0, 48.8), turned to 180 degrees
- moved C3 48.1 mm to (3.25, 25.0), turned to 270 degrees
- moved R27 46.2 mm to (4.25, 44.2), flipped to the top, turned to 90 degrees
- moved J3 45.9 mm to (24.0, 48.5), turned to 0 degrees
- moved R9 45.0 mm to (11.2, 44.2), turned to 90 degrees
- moved U2 43.5 mm to (53.1, 25.6)
- moved C1 42.9 mm to (8.50, 28.2), turned to 270 degrees
- moved C2 40.8 mm to (6.00, 24.9), turned to 270 degrees
- moved U9 40.6 mm to (5.75, 38.2), turned to 0 degrees
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- renumbered D1 to LED0, D2 to LED1, D3 to LED2, D4 to LED3, D5 to LED4, D6 to LED5, D7 to LED6, D8 to LED7, D9 to PWR
Connections:
- removed net 1V: 1000.1, C27.1, L6.1, R22.2, TP4.3, U9.3
- removed net 1V5: 2.2K.2, C19.2, L2.2, R23.1, R43.1, TP6.3, U11.1, U7.1
- removed net AD4/SELECTMAP_D3/FPGA_HOLD: U1.47, U4.C10
- removed net AD5/SELECTMAP_D2/FPGA_WP: U1.46, U4.D10
- removed net AD6/SELECTMAP_D1/SPI_MISO/MCU_PDO: J3.1, U1.13, U1.45, U3.7, U4.B12, U6.2
- removed net AD7/SELECTMAP_D0/SPI_MOSI/PDI: J3.4, U1.12, U1.44, U3.5, U4.B11, U6.5
- removed net ALE/HWB: J2.1, R4.2, U1.43, U4.G11
- removed net DDR_A0: U12.K3, U4.B3
- removed net DDR_A1: U12.L7, U4.N1
- removed net DDR_A10: U12.H7, U4.M2
- removed net DDR_A11: U12.M7, U4.P2
- removed net DDR_A12: U12.K7, U4.M4
- removed net DDR_A13: U12.N3, U4.A5
- removed net DDR_A2: U12.L3, U4.B6
- removed net DDR_A3: U12.K2, U4.B2, U4.F4
- removed net DDR_A4: U12.L8, U4.M5
- removed net DDR_A5: U12.L2, U4.B5
- removed net DDR_A6: U12.M8, U4.N4
- removed net DDR_A7: U12.M2, U4.A2
- removed net DDR_A8: U12.N8, U4.P5
- removed net DDR_A9: U12.M3, U4.A3
- removed net DDR_BA0: U12.J2, U4.C5
- removed net DDR_BA1: U12.K8, U4.M3
- removed net DDR_BA2: U12.J3, U4.B1
- removed net DDR_CAS: U12.G3, U4.C1
- removed net DDR_CKE: U12.G9, U4.M1
- removed net DDR_CLK_N: R45.1, U12.G7, U4.P3
- removed net DDR_CLK_P: R45.2, U12.F7, U4.P4
- removed net DDR_CS: U12.H2, U4.C3
- removed net DDR_DQ0: U12.B3, U4.E2
- removed net DDR_DQ1: U12.C7, U4.L2
- removed net DDR_DQ2: U12.C2, U4.E4
- removed net DDR_DQ3: U12.C8, U4.L1
- removed net DDR_DQ4: U12.E3, U4.D2
- removed net DDR_DQ5: U12.E8, U4.L3
- removed net DDR_DQ6: U12.D2, U4.D1
- removed net DDR_DQ7: U12.E7, U4.L5
- removed net DDR_DQS_N: U12.D3, U4.F1
- removed net DDR_DQS_P: U12.C3, U4.G1
- removed net DDR_ODT: U12.G1, U4.D4
- removed net DDR_RAS: U12.F3, U4.D3
- removed net DDR_RESET: U12.N2, U4.A4
- removed net DDR_WE: U12.H3, U4.C4
- removed net FPGA_VCCIO: C12.1, C15.1, C6.1, C9.1, M3.5, M3.6, M3.7, M3.8, R17.1, R18.1, R20.1, U4.G13, U4.K13, U4.N13, U4.N6, U4.N8, U7.4
- removed net FPGA_VCCIO_MON: M3.1, M3.2, M3.3
- removed net MCU_GPIO_4: J4.5, U1.15
- removed net MCU_GPIO_5: J4.6, U1.14
- removed net MCU_RX: J1.3, U1.27
- removed net MCU_TX: J1.1, U1.28
- removed net MODE2: R16.2, S3.3, U4.M9
- removed net N$18: U4.B10
- removed net N$37: U4.H14
- removed net N$4: C2.1, U1.23, X1.1
- removed net N$43: U4.F3
- removed net N$44: U4.F2
- removed net N$5: C2.2, C3.2
- removed net N$52: U4.H4
- removed net N$53: 1000.2, R39.1, U14.1
- removed net N$54: R37.1, R38.2, U14.8
- removed net N$55: L6.2, U14.4
- removed net N$56: L5.1, U14.6
- removed net N$57: D10.2, R40.2
- removed net N$58: U4.C12
- removed net N$59: U4.H3
- removed net N$6: C3.1, U1.24, X1.3
- removed net N$60: U4.H2
- removed net N$61: U4.H1
- removed net N$62: U4.J2
- removed net N$63: U4.J1
- removed net N$64: U4.K4
- removed net N$65: U4.K3
- removed net N$66: U4.J4
- removed net N$67: U4.J3
- removed net N$69: R44.1, U12.H8
- removed net N$9: U1.10
- removed net OSC_100: U4.G4, X4.3
- removed net SPI_CS: R19.2, U2.14, U4.C11, U4.L14, U6.1
- removed net SPI_SCK/CCLK: J3.3, U1.11, U3.6, U4.A8, U6.6
- removed net UID: J6.4, U1.9
- removed net VCC_DDR: R23.2, R41.2, R43.2, U11.2, U12.A2, U12.A9, U12.B9, U12.C1, U12.D7, U12.E2, U12.E9, U12.G2, U12.G8, U12.K1, U12.K9, U12.M1, U12.M9, U4.G2, U4.K2, U4.N2, U7.2, X4.1, X4.4
- removed net VREF_DDR: R41.1, R42.2, U12.E1, U12.J8
- new net AD4/SELECTMAP_D3: U1.47, U4.46
- new net AD5/SELECTMAP_D2/FPGA_MISO3: U1.46, U4.61, U5.7
- new net AD6/SELECTMAP_D1/FPGA_MISO2: U1.45, U4.62, U5.3
- new net AD7/SELECTMAP_D0/FPGA_MISO1: U1.44, U4.65, U5.2
- new net ALE: U1.43, U4.66
- new net CCLK: U1.26, U4.70, U5.6
- new net CSI_B/FPGA_MISO0: U1.25, U4.64, U5.5
- new net CSO_B: R14.2, U4.38, U5.1
- new net D+: R33.2, U11.4
- new net D-: R34.2, U11.3
- new net FTDI_RXLED: R27.1, U9.14
- new net MCU_FLASH_CE: R2.2, U1.14, U2.1
- new net MCU_MISO: U1.13, U2.2, U3.7
- new net MCU_MOSI: U1.12, U2.5, U3.5
- new net MCU_RX0/PDI: J1.4, U1.2
- new net MCU_RX1: U1.27, U9.1
- new net MCU_SCK: J1.3, U1.11, U2.6, U3.6
- new net MCU_TX0/PDO: J1.1, U1.3
- new net MCU_TX1: U1.28, U9.5
- new net MON_HWB: 15K.1, J6.1, U11.33
- new net MON_MISO: J10.1, U11.11
- new net MON_MOSI: J10.4, U11.10
- new net MON_RESET: J10.5, R35.1, S4.2, U11.13
- new net MON_SCK: J10.3, U11.9
- new net MON_VCC: 15K.2, J10.2, R16.1, R35.2, U11.14, U11.24, U11.34, U11.44, U6.10, U6.4, U7.10, U8.10
- new net MON_XTAL1: C33.1, U11.17, X4.1
- new net MON_XTAL2: C34.1, U11.16, X4.3
- new net N$14: R27.2, RX.2
- new net UCAP: C32.1, U11.6
- new net USB2_VCC: J9.1, U11.2, U11.7
- new net USB_VCC: C26.2, C27.2, L1.2, R18.2, U6.2
- new net XTAL1: C36.1, U1.24, X1.1
- new net XTAL2: C35.1, U1.23, X1.3
- net 1V2: now also C31.2, L3.2, R17.2, R31.2, U7.3; no longer C26.2, L5.2, R25.2, R37.2, TP3.3, U9.1
- net 3V3: now also C29.1, J1.2, L2.1, R16.2, R19.2, R22.2, R24.2, R25.1, R28.1, R36.1, U7.1; no longer C17.1, J3.2, L1.1, R19.1, R20.2, R21.2, R24.1, R29.2, R30.1, R31.1, TP2.3, U11.10, U14.7, U6.7, U6.8, U7.10, U7.3, U8.10, U9.10
- net 5V: now also C30.1, R18.1, RX.1, TX.1, U6.1, U9.20, U9.4; no longer C18.1, C28.1, D10.1, R36.1, TP1.3, U11.4, U14.2, U14.3, U14.5
- net A10: now also U4.81; no longer U4.E13
- net A11: now also U4.80; no longer U4.D13
- net A12: now also U4.79; no longer U4.G14
- net A13: now also U4.78; no longer U4.F14
- net A14: now also U4.75; no longer U4.F13
- net A15: now also U4.74; no longer U4.F12
- net A8: now also U4.83; no longer U4.E12
- net A9: now also U4.82; no longer U4.D12
- net AD0/SELECTMAP_D7: now also U4.48; no longer U4.B14
- net AD1/SELECTMAP_D6: now also U4.43; no longer U4.B13
- net AD2/SELECTMAP_D5/MCU_RX1: now also U4.44; no longer U4.A13
- net AD3/SELECTMAP_D4/MCU_TX1: now also U4.45; no longer U4.A12
- net ENABLE_LEDS: now also S3.3, U1.9; no longer U2.9
- net FPGA_DONE: now also U1.8, U4.71; no longer U2.8, U4.P9
- net FPGA_GPIO_0: now also U4.1; no longer U4.P13
- net FPGA_GPIO_1: now also U4.2; no longer U4.P12
- net FPGA_GPIO_10: now also U4.15; no longer U4.M10
- net FPGA_GPIO_11: now also U4.14; no longer U4.L13
- net FPGA_GPIO_12: now also U4.17; no longer U4.K12
- net FPGA_GPIO_13: now also U4.16; no longer U4.K11
- net FPGA_GPIO_14: now also U4.21; no longer U4.J14
- net FPGA_GPIO_15: now also U4.22; no longer U4.J13
- net FPGA_GPIO_16: now also U4.23; no longer U4.J12
- net FPGA_GPIO_17: now also U4.24; no longer U4.J11
- net FPGA_GPIO_18: now also U4.27
- net FPGA_GPIO_19: now also U4.26
- net FPGA_GPIO_2: now also U4.5; no longer U4.P11
- net FPGA_GPIO_3: now also U4.6; no longer U4.P10
- net FPGA_GPIO_4: now also U4.7; no longer U4.N14
- net FPGA_GPIO_5: now also U4.8; no longer U4.N11
- net FPGA_GPIO_6: now also U4.9; no longer U4.N10
- net FPGA_GPIO_7: now also U4.10; no longer U4.M14
- net FPGA_GPIO_8: now also U4.11; no longer U4.M12
- net FPGA_GPIO_9: now also U4.12; no longer U4.M11
- net FPGA_LED0: now also R8.1, U4.105; no longer R11.1
- net FPGA_LED1: now also R9.1, U4.104; no longer R12.1
- net FPGA_LED2: now also R10.1, U4.102; no longer R13.1
- net FPGA_LED3: now also R11.1, U4.101; no longer R14.1
- net FPGA_POWER: now also U1.5; no longer M3.4, U2.5
- net FPGA_RESET: now also U1.59, U4.37; no longer U2.59, U4.L7
- net FPGA_SUSPEND: now also U1.7, U4.73; no longer U2.7
- net FPGA_VCCAUX: now also C10.1, C12.1, C15.1, C16.1, C17.1, C18.1, C19.1, C2.1, C20.1, C21.1, C22.1, C23.1, C24.1, C3.1, C4.1, C6.1, C7.1, J3.1, R12.1, R13.1, R14.1, U4.103, U4.122, U4.125, U4.129, U4.135, U4.18, U4.20, U4.31, U4.36, U4.4, U4.42, U4.53, U4.63, U4.76, U4.86, U4.90, U5.8; no longer C5.1, R10.2, R16.1, U4.F10, U4.H10, U4.K10, U4.L9, U4.N7
- net FPGA_VCCAUX_MON: now also R19.1, U7.2; no longer R25.1, U9.2
- net FPGA_VCCINT: now also C1.1, C5.1, C9.1, J4.1, U4.128, U4.19, U4.28, U4.52, U4.89; no longer C10.1, C16.1, C4.1, C7.1, U4.D6, U4.D8, U4.E5, U4.E7, U4.E9, U4.F6, U4.G5, U4.G9, U4.H6, U4.J5, U4.J9, U4.K6, U4.K8
- net FPGA_VCCINT_MON: now also R17.1, U7.4; no longer R22.1, U9.4
- net GND: now also C19.2, C2.2, C20.2, C21.2, C22.2, C23.2, C24.2, C25.2, C27.1, C29.2, C3.2, C30.2, C31.1, C32.2, C33.2, C34.2, C35.2, C36.2, J1.6, J10.6, J3.3, J4.3, J6.3, J8.5, J9.5, R20.1, R21.1, R23.1, R29.2, R30.1, R32.1, S4.1, U1.53, U11.15, U11.23, U11.35, U11.43, U11.45, U2.4, U4.108, U4.113, U4.13, U4.130, U4.136, U4.25, U4.3, U4.47, U4.49, U4.54, U4.68, U4.77, U4.91, U4.96, U5.4, U6.5, U6.P$1, U6.P$2, U6.P$3, U6.P$4, U9.18, U9.21, U9.25, U9.26, U9.7; no longer C19.1, C27.2, J2.2, J3.6, J6.5, R26.1, R27.1, R28.1, R32.2, R33.1, R34.1, R35.1, R38.1, R39.2, R40.1, R42.1, R44.2, TP5.3, U1.6, U11.P$1, U11.P$2, U11.P$3, U11.P$4, U12.A1, U12.A8, U12.B1, U12.B2, U12.B7, U12.B8, U12.C9, U12.D1, U12.D8, U12.D9, U12.F2, U12.F8, U12.J1, U12.J9, U12.L1, U12.L9, U12.N1, U12.N9, U14.9, U4.A1, U4.A11, U4.A14, U4.A6, U4.A9, U4.B4, U4.B7, U4.B9, U4.C13, U4.C2, U4.C6, U4.C7, U4.C8, U4.C9, U4.D11, U4.D5, U4.D7, U4.D9, U4.E1, U4.E10, U4.E14, U4.E3, U4.E6, U4.E8, U4.F5, U4.F9, U4.G10, U4.G12, U4.G3, U4.G6, U4.H5, U4.H9, U4.J10, U4.J6, U4.J7, U4.J8, U4.K1, U4.K14, U4.K5, U4.K7, U4.K9, U4.L10, U4.L11, U4.L12, U4.L4, U4.L6, U4.L8, U4.M13, U4.N12, U4.N3, U4.N5, U4.N9, U4.P1, U4.P14, U6.4, U9.5, U9.P$1, U9.P$2, U9.P$3, U9.P$4, X4.2
- net INIT_B: now also U1.58, U4.39; no longer R10.1, U2.58, U4.P8
- net JTAG_TCK: now also U4.109; no longer U4.A7
- net JTAG_TDI: now also U1.55, U4.110; no longer U1.54, U4.P7
- net JTAG_TDO: now also U1.56, U4.106; no longer U1.55, U4.P6
- net JTAG_TMS: now also U1.54, U4.107; no longer U1.56, U4.M6
- net MCU_GPIO_0: now also J2.1, U1.17; no longer J4.1, U1.19
- net MCU_GPIO_1: now also J2.2; no longer J4.2
- net MCU_GPIO_2: now also J2.3, U1.19; no longer J4.3, U1.17
- net MCU_GPIO_3: now also J2.4; no longer J4.4
- net MCU_LED0: now also R3.1, U1.32; no longer R5.1, U2.32
- net MCU_LED1: now also R4.1, U1.31; no longer R6.1, U2.31
- net MCU_LED2: now also R5.1, U1.30; no longer R7.1, U2.30
- net MCU_LED3: now also R6.1, U1.29; no longer R8.1, U2.29
- net MCU_RESET: now also J1.5, R7.1; no longer J3.5, R9.1
- net MCU_VCC: now also R1.1, R2.1, R22.1, R7.2, U2.3, U2.7, U2.8; no longer C1.1, R21.1, R3.1, R4.1, R9.2, U1.3, U1.53, U1.7
- net MODE0: now also R12.2, U4.69; no longer R18.2, U4.M7
- net MODE1: now also R13.2, U4.60; no longer R17.2, U4.M8
- net MONITORING: now also U11.1
- net N$1: now also L2.2; no longer L1.2
- net N$10: now also R26.1, U9.13; no longer R1.2, U1.5
- net N$11: now also R26.2, TX.2; no longer R35.2, U11.6
- net N$13: now also R6.2; no longer R8.2
- net N$15: now also R5.2; no longer R7.2
- net N$16: now also R23.2; no longer R27.2
- net N$2: now also R28.2, R29.1; no longer R31.2, R32.1
- net N$23: now also R4.2; no longer R6.2
- net N$24: now also R3.2; no longer R5.2
- net N$25: now also R11.2; no longer R14.2
- net N$27: now also R10.2; no longer R13.2
- net N$28: now also R21.2, U7.6; no longer R28.2, U9.6
- net N$29: now also R9.2; no longer R12.2
- net N$3: now also C28.1, U9.17; no longer R2.2, U1.4
- net N$30: now also R8.2; no longer R11.2
- net N$32: now also R20.2, U6.6; no longer R26.2, U7.6
- net N$38: now also J9.3, R33.1; no longer U4.H13
- net N$39: now also J9.2, R34.1; no longer U4.H12
- net N$41: now also R32.2; no longer R33.2
- net N$7: now also R30.2, R31.1; no longer 2.2K.1, R34.2
- net N$8: now also L3.1; no longer L2.1
- net OSC_32: now also U4.94; no longer U4.H11
- net OSC_50: now also U4.51; no longer U4.F11
- net RD: now also U4.84; no longer U4.C14
- net SCL: now also R24.1, U11.18, U6.9; no longer R29.1, U1.25, U11.9, U9.9
- net SDA: now also R25.2, U11.19, U6.8; no longer R30.2, U1.26, U11.8, U9.8
- net USBD+: now also J8.3, U9.15; no longer J6.3, R1.1
- net USBD-: now also J8.2, U9.16; no longer J6.2, R2.1
- net USB_VCC_RAW: now also C25.1, J8.1, L1.1; no longer J6.1, R36.2, U1.8, U11.3
- net WIRELESS_CS: now also R1.2, U1.60; no longer R3.2, U2.60
- net WIRELESS_INT: now also U1.61; no longer U2.61
- net WIRELESS_RESET: now also U1.15; no longer U2.15
- net WIRELESS_VCC: now also R36.2; no longer R24.2
- net WIRELESS_WAKE: now also U1.4; no longer U2.4
- net WR: now also U4.85; no longer U4.D14
Routing:
- net FPGA_VCCAUX: track 0.00 -> 266.1 mm, vias 0 -> 16
- net MON_VCC: track 0.00 -> 190.6 mm, vias 0 -> 7
- net 3V3: track 0.00 -> 128.4 mm, vias 0 -> 12
- net FPGA_VCCINT: track 0.00 -> 104.9 mm, vias 0 -> 5
- net GND: track 0.00 -> 84.9 mm, vias 0 -> 63
- net SDA: track 0.00 -> 81.4 mm, vias 0 -> 3
- net SCL: track 0.00 -> 73.2 mm
- net MCU_VCC: track 0.00 -> 67.4 mm, vias 0 -> 8
- net 5V: track 0.00 -> 63.4 mm, vias 0 -> 6
- net MCU_SCK: track 0.00 -> 56.7 mm, vias 0 -> 4
- net MON_RESET: track 0.00 -> 48.1 mm, vias 0 -> 2
- net MCU_MISO: track 0.00 -> 47.7 mm, vias 0 -> 3
- net MONITORING: track 0.00 -> 45.5 mm, vias 0 -> 3
- net MCU_RESET: track 0.00 -> 44.2 mm, vias 0 -> 2
- net MCU_MOSI: track 0.00 -> 42.4 mm, vias 0 -> 1
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- added copper zone on layer 16, net 1V2
- removed copper zone on layer 16, net 1V
Other:
- board text removed: "58,25 52,5"
